File: eagle/NinjaFuge-DIP-171003.brd (EAGLE design)
At the start: 81.7 x 23.7 mm, 22 parts, among them IC1 2x14p-2.54, IC2 7805TV

Commit message: added another reed to check lock is locked or just hitting the wall
Parts:
- R4: value 500 -> 330
- R5: value 160 -> 100
Changed lines of the file:
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@@
 <attribute name="VALUE" x="76.095" y="19.349" size="1.27" layer="28" ratio="10" rot="MR0"/>
 </element>
-<element name="R4" library="rcl" package="0204/5" value="500" x="57.7" y="22.4" smashed="yes">
+<element name="R4" library="rcl" package="0204/5" value="330" x="57.7" y="22.4" smashed="yes">
 <attribute name="NAME" x="56.7602" y="21.9682" size="0.9906" layer="25" ratio="10"/>
 </element>
@@
 <attribute name="VALUE" x="68.095" y="19.349" size="1.27" layer="28" ratio="10" rot="MR0"/>
 </element>
-<element name="R5" library="rcl" package="0204/5" value="160" x="57.7" y="20.4" smashed="yes">
+<element name="R5" library="rcl" package="0204/5" value="100" x="57.7" y="20.4" smashed="yes">
 <attribute name="NAME" x="56.7094" y="19.9682" size="0.9906" layer="25" ratio="10"/>
 </element>
